File: Hardware/AngelCarol.kicad_sch (KiCad schematic)
At the start: 32 parts, among them J1 COIN_DET, J2 SPEAKER, J3 POWER, J4 OUT, J5 SWD, Q1 BC817, Q2 BC817, Q3 IRLML5203, U1 STM32C011F6Px

Commit message: Tune some components values, add PK handler model
Parts:
- C1: value 100nF -> 4.7u
- R2: value 47k -> 4k7
- R3: value 10k -> 470
- R5, R6: value 10k -> 2k2
- R7, R8: value 10k -> 33k
- R9: value 10k -> 1k
Changed lines of the file:
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@@
 			)
 		)
-		(property "Value" "10k"
+		(property "Value" "470"
 			(at 233.68 35.5599 0)
 			(effects
@@
 			)
 		)
-		(property "Value" "10k"
+		(property "Value" "33k"
 			(at 73.66 133.3499 0)
 			(effects
@@
 			)
 		)
-		(property "Value" "10k"
+		(property "Value" "33k"
 			(at 73.66 109.2199 0)
 			(effects
@@
 			)
 		)
-		(property "Value" "47k"
+		(property "Value" "4k7"
 			(at 203.2 35.5599 0)
 			(effects
@@
 			)
 		)
-		(property "Value" "10k"
+		(property "Value" "1k"
 			(at 152.4 115.57 90)
 			(effects
@@
 			)
 		)
-		(property "Value" "100nF"
+		(property "Value" "4.7u"
 			(at 248.92 116.8399 0)
 			(effects
@@
 			)
 		)
-		(property "Value" "10k"
+		(property "Value" "2k2"
 			(at 76.2 121.92 90)
 			(effects
@@
 			)
 		)
-		(property "Value" "10k"
+		(property "Value" "2k2"
 			(at 76.2 97.79 90)
 			(effects

Commit message: Some fix in schematic
Connections:
- net COIN_DET_SIG: now also U1.10 (PA3); no longer U1.3 (PC15)
Changed lines of the file:
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@@
+	)
+	(no_connect
+		(at 111.76 99.06)
+	)
+	(no_connect
+		(at 227.33 120.65)
+	)
+	(no_connect
+		(at 139.7 104.14)
+	)
+	(no_connect
+		(at 111.76 111.76)
+	)
+	(no_connect
+		(at 227.33 107.95)
+	)
+	(no_connect
+		(at 72.39 49.53)
 	)
 	(no_connect
@@
 	)
 	(no_connect
-		(at 111.76 99.06)
-	)
-	(no_connect
-		(at 227.33 120.65)
-	)
-	(no_connect
-		(at 139.7 104.14)
-	)
-	(no_connect
-		(at 111.76 111.76)
-	)
-	(no_connect
-		(at 227.33 107.95)
-	)
-	(no_connect
-		(at 72.39 49.53)
-	)
-	(no_connect
-		(at 139.7 106.68)
-	)
-	(no_connect
 		(at 227.33 118.11)
 	)
@@
 	)
 	(no_connect
+		(at 111.76 106.68)
+	)
+	(no_connect
 		(at 227.33 125.73)
 	)
@@
 	(global_label "COIN_DET_SIG"
 		(shape input)
-		(at 111.76 106.68 180)
-		(fields_autoplaced yes)
-		(effects
-			(font
-				(size 1.27 1.27)
-			)
-			(justify right)
-		)
-		(property "Intersheetrefs" "${INTERSHEET_REFS}"
-			(at 95.8329 106.68 0)
-			(effects
-				(font
-					(size 1.27 1.27)
-				)
-				(justify right)
-				(hide yes)
-			)
+		(at 139.7 106.68 0)
+		(fields_autoplaced yes)
+		(effects
+			(font
+				(size 1.27 1.27)
+			)
+			(justify left)
+		)
+		(property "Intersheetrefs" "${INTERSHEET_REFS}"
+			(at 155.6271 106.68 0)
+			(effects
+				(font
+					(size 1.27 1.27)
+				)
+				(justify left)
+				(hide yes)
+			)
